File: MAX17048/MAX17048.sch (KiCad schematic (older format))
At the start: 4 parts

Commit message: Update schematics
Parts:
- gave numbers to parts that had none: 4
Changed lines of the file:
@@
 $Descr A4 11693 8268
 encoding utf-8
-Sheet 6 6
+Sheet 5 6
 Title ""
 Date ""
@@
 AR Path="/5F610235/5F260DCC" Ref="R?"  Part="1"
 AR Path="/5F6110E7/5F260DCC" Ref="R?"  Part="1"
-AR Path="/5F61393C/5F260DCC" Ref="R?"  Part="1"
-F 0 "R?" H 3920 3846 50  0000 L CNN
+AR Path="/5F61393C/5F260DCC" Ref="R16"  Part="1"
+F 0 "R16" H 3920 3846 50  0000 L CNN
 F 1 "R" H 3920 3755 50  0000 L CNN
 F 2 "" V 3780 3800 50  0001 C CNN
@@
 AR Path="/5F610235/5F2610AB" Ref="R?"  Part="1"
 AR Path="/5F6110E7/5F2610AB" Ref="R?"  Part="1"
-AR Path="/5F61393C/5F2610AB" Ref="R?"  Part="1"
-F 0 "R?" H 3920 4346 50  0000 L CNN
+AR Path="/5F61393C/5F2610AB" Ref="R17"  Part="1"
+F 0 "R17" H 3920 4346 50  0000 L CNN
 F 1 "R" H 3920 4255 50  0000 L CNN
 F 2 "" V 3780 4300 50  0001 C CNN
@@
 AR Path="/5F610235/5F262B46" Ref="#PWR?"  Part="1"
 AR Path="/5F6110E7/5F262B46" Ref="#PWR?"  Part="1"
-AR Path="/5F61393C/5F262B46" Ref="#PWR?"  Part="1"
-F 0 "#PWR?" H 3850 4300 50  0001 C CNN
+AR Path="/5F61393C/5F262B46" Ref="#PWR084"  Part="1"
+F 0 "#PWR084" H 3850 4300 50  0001 C CNN
 F 1 "GND" H 3855 4377 50  0000 C CNN
 F 2 "" H 3850 4550 50  0001 C CNN
@@
 AR Path="/5F610235/5F266736" Ref="C?"  Part="1"
 AR Path="/5F6110E7/5F266736" Ref="C?"  Part="1"
-AR Path="/5F61393C/5F266736" Ref="C?"  Part="1"
-F 0 "C?" H 4365 4346 50  0000 L CNN
+AR Path="/5F61393C/5F266736" Ref="C15"  Part="1"
+F 0 "C15" H 4365 4346 50  0000 L CNN
 F 1 "0.1u" H 4365 4255 50  0000 L CNN
 F 2 "" H 4288 4150 50  0001 C CNN
@@
 AR Path="/5F610235/5F266DAF" Ref="#PWR?"  Part="1"
 AR Path="/5F6110E7/5F266DAF" Ref="#PWR?"  Part="1"
-AR Path="/5F61393C/5F266DAF" Ref="#PWR?"  Part="1"
-F 0 "#PWR?" H 4250 4300 50  0001 C CNN
+AR Path="/5F61393C/5F266DAF" Ref="#PWR085"  Part="1"
+F 0 "#PWR085" H 4250 4300 50  0001 C CNN
 F 1 "GND" H 4255 4377 50  0000 C CNN
 F 2 "" H 4250 4550 50  0001 C CNN
@@
 AR Path="/5F610235/5F2672F0" Ref="#PWR?"  Part="1"
 AR Path="/5F6110E7/5F2672F0" Ref="#PWR?"  Part="1"
-AR Path="/5F61393C/5F2672F0" Ref="#PWR?"  Part="1"
-F 0 "#PWR?" H 4650 4300 50  0001 C CNN
+AR Path="/5F61393C/5F2672F0" Ref="#PWR086"  Part="1"
+F 0 "#PWR086" H 4650 4300 50  0001 C CNN
 F 1 "GND" H 4655 4377 50  0000 C CNN
 F 2 "" H 4650 4550 50  0001 C CNN
@@
 AR Path="/5F610235/5F26E3EE" Ref="#PWR?"  Part="1"
 AR Path="/5F6110E7/5F26E3EE" Ref="#PWR?"  Part="1"
-AR Path="/5F61393C/5F26E3EE" Ref="#PWR?"  Part="1"
-F 0 "#PWR?" H 7650 4350 50  0001 C CNN
+AR Path="/5F61393C/5F26E3EE" Ref="#PWR087"  Part="1"
+F 0 "#PWR087" H 7650 4350 50  0001 C CNN
 F 1 "GND" H 7655 4427 50  0000 C CNN
 F 2 "" H 7650 4600 50  0001 C CNN
@@
 NoConn ~ 7300 3950
 $Comp
-L max17048:MAX17048G+ U?
+L max17048:MAX17048G+ U6
 U 1 1 5F7BC92F
 P 4900 3950
-F 0 "U?" H 6100 4337 60  0000 C CNN
+F 0 "U6" H 6100 4337 60  0000 C CNN
 F 1 "MAX17048G+" H 6100 4231 60  0000 C CNN
 F 2 "21-0168E_T822-3_MXM" H 6100 4190 60  0001 C CNN

Commit message: Cleanup #1
Parts:
- U6: symbol max17048:MAX17048G+ -> core-rescue:MAX17048G+-max17048
Changed lines of the file:
@@
 NoConn ~ 7300 3950
 $Comp
-L max17048:MAX17048G+ U6
+L core-rescue:MAX17048G+-max17048 U6
 U 1 1 5F7BC92F
 P 4900 3950
+AR Path="/5F7BC92F" Ref="U6"  Part="1"
+AR Path="/5F61393C/5F7BC92F" Ref="U6"  Part="1"
 F 0 "U6" H 6100 4337 60  0000 C CNN
 F 1 "MAX17048G+" H 6100 4231 60  0000 C CNN

Commit message: Fixed broken symbols
Parts:
- removed U6: MAX17048G+, 21-0168E_T822-3_MXM, symbol core-rescue:MAX17048G+-max17048
- added U?: MAX17048G+, 21-0168E_T822-3_MXM, symbol star-common-lib:MAX17048G+
Changed lines of the file:
@@
 NoConn ~ 7300 3950
 $Comp
-L core-rescue:MAX17048G+-max17048 U6
-U 1 1 5F7BC92F
+L star-common-lib:MAX17048G+ U?
+U 1 1 5F61DB0A
 P 4900 3950
-AR Path="/5F7BC92F" Ref="U6"  Part="1"
-AR Path="/5F61393C/5F7BC92F" Ref="U6"  Part="1"
-F 0 "U6" H 6100 4337 60  0000 C CNN
-F 1 "MAX17048G+" H 6100 4231 60  0000 C CNN
+F 0 "U?" H 6100 4443 60  0000 C CNN
+F 1 "MAX17048G+" H 6100 4337 60  0000 C CNN
 F 2 "21-0168E_T822-3_MXM" H 6100 4190 60  0001 C CNN
-F 3 "" H 4900 3950 60  0000 C CNN
+F 3 "https://datasheets.maximintegrated.com/en/ds/MAX17048-MAX17049.pdf" H 6100 4231 60  0000 C CNN
 	1    4900 3950
 	1    0    0    -1
