File: BNO055/BNO055.sch (KiCad schematic (older format))
At the start: 9 parts, among them U4 BNO055

Commit message: add fields, pick components, and add footprints
Parts:
- removed R10, R11: 10k, Resistor_SMD:R_0603_1608Metric, symbol Device:R
- C1201: renamed from C20; DIGIKEY (none) -> 399-1100-1-ND; MANF (none) -> C0603C104Z3VACTU
- C1202: renamed from C17; DIGIKEY (none) -> 1292-1459-1-ND; MANF (none) -> 0603B682K500CT
- C1203: renamed from C18; DIGIKEY (none) -> 311-4056-1-ND; MANF (none) -> CC0603KRX7R6BB124
- C1204: renamed from C19; DIGIKEY (none) -> 399-1100-1-ND; MANF (none) -> C0603C104Z3VACTU
- R1201: renamed from R9; DIGIKEY (none) -> 311-10KGRCT-ND; MANF (none) -> RC0603JR-0710KL
- R1202: renamed from R8; DIGIKEY (none) -> 311-10KGRCT-ND; MANF (none) -> RC0603JR-0710KL
- U1201: renamed from U4; DIGIKEY (none) -> 828-1058-1-ND; MANF (none) -> BNO055
Connections:
- wire segments 60 -> 36
Other:
- moved on the sheet: C1202, C1203, C1204, R1201, R1202
