File: BNO055/BNO055.sch (KiCad schematic (older format))
At the start: 9 parts, among them U4 BNO055

Commit message: Update Schematic blocks
Parts:
- renumbered C20 to C10, C17 to C7, C18 to C8, C19 to C9, R8 to R4, R9 to R5, R10 to R6, R11 to R7, U4 to U3
Connections:
- wire segments 60 -> 56
Changed lines of the file:
@@
 $Descr A4 11693 8268
 encoding utf-8
-Sheet 4 5
+Sheet 2 6
 Title ""
 Date ""
@@
 P 5900 4000
 AR Path="/5E6B3267" Ref="U?"  Part="1"
-AR Path="/5E6B2FC0/5E6B3267" Ref="U4"  Part="1"
-F 0 "U4" H 6200 4900 50  0000 C CNN
+AR Path="/5E6B2FC0/5E6B3267" Ref="U3"  Part="1"
+F 0 "U3" H 6200 4900 50  0000 C CNN
 F 1 "BNO055" H 6200 4800 50  0000 C CNN
 F 2 "Package_LGA:LGA-28_5.2x3.8mm_P0.5mm" H 6150 3350 50  0001 L CNN
@@
 P 6900 4750
 AR Path="/5E6B326E" Ref="#PWR?"  Part="1"
-AR Path="/5E6B2FC0/5E6B326E" Ref="#PWR03"  Part="1"
-F 0 "#PWR03" H 6900 4500 50  0001 C CNN
+AR Path="/5E6B2FC0/5E6B326E" Ref="#PWR028"  Part="1"
+F 0 "#PWR028" H 6900 4500 50  0001 C CNN
 F 1 "GND" H 6905 4577 50  0000 C CNN
 F 2 "" H 6900 4750 50  0001 C CNN
@@
 P 6750 4500
 AR Path="/5E6B3274" Ref="C?"  Part="1"
-AR Path="/5E6B2FC0/5E6B3274" Ref="C20"  Part="1"
-F 0 "C20" V 6700 4350 50  0000 C CNN
+AR Path="/5E6B2FC0/5E6B3274" Ref="C10"  Part="1"
+F 0 "C10" V 6700 4350 50  0000 C CNN
 F 1 "100nF" V 6800 4350 50  0000 C CNN
 F 2 "Capacitor_SMD:C_0603_1608Metric" H 6788 4350 50  0001 C CNN
@@
 	5800 4750 5800 4700
 Wire Wire Line
-	6200 4700 6200 4750
-Wire Wire Line
-	6100 4700 6100 4750
-Connection ~ 6100 4750
-Wire Wire Line
-	6100 4750 6200 4750
-Wire Wire Line
 	6000 4700 6000 4750
 Connection ~ 6000 4750
-Wire Wire Line
-	6000 4750 6100 4750
 Wire Wire Line
 	5300 4400 5250 4400
@@
 P 5650 5100
 AR Path="/5E6B3291" Ref="C?"  Part="1"
-AR Path="/5E6B2FC0/5E6B3291" Ref="C19"  Part="1"
-F 0 "C19" V 5600 4950 50  0000 C CNN
+AR Path="/5E6B2FC0/5E6B3291" Ref="C9"  Part="1"
+F 0 "C9" V 5600 4950 50  0000 C CNN
 F 1 "100nF" V 5700 4950 50  0000 C CNN
 F 2 "Capacitor_SMD:C_0603_1608Metric" H 5688 4950 50  0001 C CNN
@@
 P 4950 4450
 AR Path="/5E6B329F" Ref="R?"  Part="1"
-AR Path="/5E6B2FC0/5E6B329F" Ref="R11"  Part="1"
-F 0 "R11" V 4900 4250 50  0000 C CNN
+AR Path="/5E6B2FC0/5E6B329F" Ref="R7"  Part="1"
+F 0 "R7" V 4900 4250 50  0000 C CNN
 F 1 "10k" V 5000 4250 50  0000 C CNN
 F 2 "Resistor_SMD:R_0603_1608Metric" V 4880 4450 50  0001 C CNN
@@
 P 4950 4050
 AR Path="/5E6B32AB" Ref="R?"  Part="1"
-AR Path="/5E6B2FC0/5E6B32AB" Ref="R10"  Part="1"
-F 0 "R10" V 4900 3850 50  0000 C CNN
+AR Path="/5E6B2FC0/5E6B32AB" Ref="R6"  Part="1"
+F 0 "R6" V 4900 3850 50  0000 C CNN
 F 1 "10k" V 5000 3850 50  0000 C CNN
 F 2 "Resistor_SMD:R_0603_1608Metric" V 4880 4050 50  0001 C CNN
@@
 P 4900 3850
 AR Path="/5E6B32B7" Ref="R?"  Part="1"
-AR Path="/5E6B2FC0/5E6B32B7" Ref="R9"  Part="1"
-F 0 "R9" V 4850 4050 50  0000 C CNN
+AR Path="/5E6B2FC0/5E6B32B7" Ref="R5"  Part="1"
+F 0 "R5" V 4850 4050 50  0000 C CNN
 F 1 "10k" V 4950 4050 50  0000 C CNN
 F 2 "Resistor_SMD:R_0603_1608Metric" V 4830 3850 50  0001 C CNN
@@
 P 4900 3400
 AR Path="/5E6B32C1" Ref="R?"  Part="1"
-AR Path="/5E6B2FC0/5E6B32C1" Ref="R8"  Part="1"
-F 0 "R8" V 4850 3200 50  0000 C CNN
+AR Path="/5E6B2FC0/5E6B32C1" Ref="R4"  Part="1"
+F 0 "R4" V 4850 3200 50  0000 C CNN
 F 1 "10k" V 4950 3200 50  0000 C CNN
 F 2 "Resistor_SMD:R_0603_1608Metric" V 4830 3400 50  0001 C CNN
@@
 P 4900 4750
 AR Path="/5E6B32CC" Ref="C?"  Part="1"
-AR Path="/5E6B2FC0/5E6B32CC" Ref="C17"  Part="1"
-F 0 "C17" V 4850 4900 50  0000 C CNN
+AR Path="/5E6B2FC0/5E6B32CC" Ref="C7"  Part="1"
+F 0 "C7" V 4850 4900 50  0000 C CNN
 F 1 "6.8nF" V 4950 4900 50  0000 C CNN
 F 2 "Capacitor_SMD:C_0603_1608Metric" H 4938 4600 50  0001 C CNN
@@
 P 4900 4950
 AR Path="/5E6B32D3" Ref="C?"  Part="1"
-AR Path="/5E6B2FC0/5E6B32D3" Ref="C18"  Part="1"
-F 0 "C18" V 4850 4800 50  0000 C CNN
+AR Path="/5E6B2FC0/5E6B32D3" Ref="C8"  Part="1"
+F 0 "C8" V 4850 4800 50  0000 C CNN
 F 1 "120nF" V 4950 4750 50  0000 C CNN
 F 2 "Capacitor_SMD:C_0603_1608Metric" H 4938 4800 50  0001 C CNN
@@
 P 5400 5000
 AR Path="/5E6B32E9" Ref="#PWR?"  Part="1"
-AR Path="/5E6B2FC0/5E6B32E9" Ref="#PWR02"  Part="1"
-F 0 "#PWR02" H 5400 4850 50  0001 C CNN
+AR Path="/5E6B2FC0/5E6B32E9" Ref="#PWR027"  Part="1"
+F 0 "#PWR027" H 5400 4850 50  0001 C CNN
 F 1 "+3.3V" H 5400 5150 50  0000 C CNN
 F 2 "" H 5400 5000 50  0001 C CNN
@@
 P 5350 3250
 AR Path="/5E6B32F9" Ref="#PWR?"  Part="1"
-AR Path="/5E6B2FC0/5E6B32F9" Ref="#PWR01"  Part="1"
-F 0 "#PWR01" H 5350 3100 50  0001 C CNN
+AR Path="/5E6B2FC0/5E6B32F9" Ref="#PWR026"  Part="1"
+F 0 "#PWR026" H 5350 3100 50  0001 C CNN
 F 1 "+3.3V" H 5350 3400 50  0000 C CNN
 F 2 "" H 5350 3250 50  0001 C CNN
@@
 Wire Wire Line
 	5100 4450 5200 4450
-Wire Wire Line
-	6200 4750 6900 4750
-Connection ~ 6200 4750
 Wire Wire Line
 	6600 4500 6500 4500
@@
 Text Notes 7300 6900 0    118  ~ 0
 BNO055 Hierarchical Block (I2C)
+Wire Wire Line
+	6000 4750 6900 4750
 $EndSCHEMATC

Commit message: Update schematics
Parts:
- renumbered C8 to C10, C9 to C11, C10 to C12, C7 to C9, R4 to R10, R5 to R11, R6 to R12, R7 to R13, U3 to U4
Connections:
- no-connect marks 3 -> 4
Changed lines of the file:
@@
 P 5900 4000
 AR Path="/5E6B3267" Ref="U?"  Part="1"
-AR Path="/5E6B2FC0/5E6B3267" Ref="U3"  Part="1"
-F 0 "U3" H 6200 4900 50  0000 C CNN
+AR Path="/5E6B2FC0/5E6B3267" Ref="U4"  Part="1"
+F 0 "U4" H 6200 4900 50  0000 C CNN
 F 1 "BNO055" H 6200 4800 50  0000 C CNN
 F 2 "Package_LGA:LGA-28_5.2x3.8mm_P0.5mm" H 6150 3350 50  0001 L CNN
@@
 P 6900 4750
 AR Path="/5E6B326E" Ref="#PWR?"  Part="1"
-AR Path="/5E6B2FC0/5E6B326E" Ref="#PWR028"  Part="1"
-F 0 "#PWR028" H 6900 4500 50  0001 C CNN
+AR Path="/5E6B2FC0/5E6B326E" Ref="#PWR048"  Part="1"
+F 0 "#PWR048" H 6900 4500 50  0001 C CNN
 F 1 "GND" H 6905 4577 50  0000 C CNN
 F 2 "" H 6900 4750 50  0001 C CNN
@@
 P 6750 4500
 AR Path="/5E6B3274" Ref="C?"  Part="1"
-AR Path="/5E6B2FC0/5E6B3274" Ref="C10"  Part="1"
-F 0 "C10" V 6700 4350 50  0000 C CNN
+AR Path="/5E6B2FC0/5E6B3274" Ref="C12"  Part="1"
+F 0 "C12" V 6700 4350 50  0000 C CNN
 F 1 "100nF" V 6800 4350 50  0000 C CNN
 F 2 "Capacitor_SMD:C_0603_1608Metric" H 6788 4350 50  0001 C CNN
@@
 P 5650 5100
 AR Path="/5E6B3291" Ref="C?"  Part="1"
-AR Path="/5E6B2FC0/5E6B3291" Ref="C9"  Part="1"
-F 0 "C9" V 5600 4950 50  0000 C CNN
+AR Path="/5E6B2FC0/5E6B3291" Ref="C11"  Part="1"
+F 0 "C11" V 5600 4950 50  0000 C CNN
 F 1 "100nF" V 5700 4950 50  0000 C CNN
 F 2 "Capacitor_SMD:C_0603_1608Metric" H 5688 4950 50  0001 C CNN
@@
 P 4950 4450
 AR Path="/5E6B329F" Ref="R?"  Part="1"
-AR Path="/5E6B2FC0/5E6B329F" Ref="R7"  Part="1"
-F 0 "R7" V 4900 4250 50  0000 C CNN
+AR Path="/5E6B2FC0/5E6B329F" Ref="R13"  Part="1"
+F 0 "R13" V 4900 4250 50  0000 C CNN
 F 1 "10k" V 5000 4250 50  0000 C CNN
 F 2 "Resistor_SMD:R_0603_1608Metric" V 4880 4450 50  0001 C CNN
@@
 P 4950 4050
 AR Path="/5E6B32AB" Ref="R?"  Part="1"
-AR Path="/5E6B2FC0/5E6B32AB" Ref="R6"  Part="1"
-F 0 "R6" V 4900 3850 50  0000 C CNN
+AR Path="/5E6B2FC0/5E6B32AB" Ref="R12"  Part="1"
+F 0 "R12" V 4900 3850 50  0000 C CNN
 F 1 "10k" V 5000 3850 50  0000 C CNN
 F 2 "Resistor_SMD:R_0603_1608Metric" V 4880 4050 50  0001 C CNN
@@
 P 4900 3850
 AR Path="/5E6B32B7" Ref="R?"  Part="1"
-AR Path="/5E6B2FC0/5E6B32B7" Ref="R5"  Part="1"
-F 0 "R5" V 4850 4050 50  0000 C CNN
+AR Path="/5E6B2FC0/5E6B32B7" Ref="R11"  Part="1"
+F 0 "R11" V 4850 4050 50  0000 C CNN
 F 1 "10k" V 4950 4050 50  0000 C CNN
 F 2 "Resistor_SMD:R_0603_1608Metric" V 4830 3850 50  0001 C CNN
@@
 P 4900 3400
 AR Path="/5E6B32C1" Ref="R?"  Part="1"
-AR Path="/5E6B2FC0/5E6B32C1" Ref="R4"  Part="1"
-F 0 "R4" V 4850 3200 50  0000 C CNN
+AR Path="/5E6B2FC0/5E6B32C1" Ref="R10"  Part="1"
+F 0 "R10" V 4850 3200 50  0000 C CNN
 F 1 "10k" V 4950 3200 50  0000 C CNN
 F 2 "Resistor_SMD:R_0603_1608Metric" V 4830 3400 50  0001 C CNN
@@
 P 4900 4750
 AR Path="/5E6B32CC" Ref="C?"  Part="1"
-AR Path="/5E6B2FC0/5E6B32CC" Ref="C7"  Part="1"
-F 0 "C7" V 4850 4900 50  0000 C CNN
+AR Path="/5E6B2FC0/5E6B32CC" Ref="C9"  Part="1"
+F 0 "C9" V 4850 4900 50  0000 C CNN
 F 1 "6.8nF" V 4950 4900 50  0000 C CNN
 F 2 "Capacitor_SMD:C_0603_1608Metric" H 4938 4600 50  0001 C CNN
@@
 P 4900 4950
 AR Path="/5E6B32D3" Ref="C?"  Part="1"
-AR Path="/5E6B2FC0/5E6B32D3" Ref="C8"  Part="1"
-F 0 "C8" V 4850 4800 50  0000 C CNN
+AR Path="/5E6B2FC0/5E6B32D3" Ref="C10"  Part="1"
+F 0 "C10" V 4850 4800 50  0000 C CNN
 F 1 "120nF" V 4950 4750 50  0000 C CNN
 F 2 "Capacitor_SMD:C_0603_1608Metric" H 4938 4800 50  0001 C CNN
@@
 P 5400 5000
 AR Path="/5E6B32E9" Ref="#PWR?"  Part="1"
-AR Path="/5E6B2FC0/5E6B32E9" Ref="#PWR027"  Part="1"
-F 0 "#PWR027" H 5400 4850 50  0001 C CNN
+AR Path="/5E6B2FC0/5E6B32E9" Ref="#PWR047"  Part="1"
+F 0 "#PWR047" H 5400 4850 50  0001 C CNN
 F 1 "+3.3V" H 5400 5150 50  0000 C CNN
 F 2 "" H 5400 5000 50  0001 C CNN
@@
 P 5350 3250
 AR Path="/5E6B32F9" Ref="#PWR?"  Part="1"
-AR Path="/5E6B2FC0/5E6B32F9" Ref="#PWR026"  Part="1"
-F 0 "#PWR026" H 5350 3100 50  0001 C CNN
+AR Path="/5E6B2FC0/5E6B32F9" Ref="#PWR046"  Part="1"
+F 0 "#PWR046" H 5350 3100 50  0001 C CNN
 F 1 "+3.3V" H 5350 3400 50  0000 C CNN
 F 2 "" H 5350 3250 50  0001 C CNN
@@
 Wire Wire Line
 	6000 4750 6900 4750
+NoConn ~ 7350 4700
 $EndSCHEMATC

Commit message: Revert schematics so that it can merge
Parts:
- renumbered C9 to C17, C10 to C18, C11 to C19, C12 to C20, R12 to R10, R13 to R11, R10 to R8, R11 to R9
Connections:
- wire segments 56 -> 60
- no-connect marks 4 -> 3
Changed lines of the file:
@@
 $Descr A4 11693 8268
 encoding utf-8
-Sheet 2 6
+Sheet 4 6
 Title ""
 Date ""
@@
 P 6900 4750
 AR Path="/5E6B326E" Ref="#PWR?"  Part="1"
-AR Path="/5E6B2FC0/5E6B326E" Ref="#PWR048"  Part="1"
-F 0 "#PWR048" H 6900 4500 50  0001 C CNN
+AR Path="/5E6B2FC0/5E6B326E" Ref="#PWR03"  Part="1"
+F 0 "#PWR03" H 6900 4500 50  0001 C CNN
 F 1 "GND" H 6905 4577 50  0000 C CNN
 F 2 "" H 6900 4750 50  0001 C CNN
@@
 P 6750 4500
 AR Path="/5E6B3274" Ref="C?"  Part="1"
-AR Path="/5E6B2FC0/5E6B3274" Ref="C12"  Part="1"
-F 0 "C12" V 6700 4350 50  0000 C CNN
+AR Path="/5E6B2FC0/5E6B3274" Ref="C20"  Part="1"
+F 0 "C20" V 6700 4350 50  0000 C CNN
 F 1 "100nF" V 6800 4350 50  0000 C CNN
 F 2 "Capacitor_SMD:C_0603_1608Metric" H 6788 4350 50  0001 C CNN
@@
 	5800 4750 5800 4700
 Wire Wire Line
+	6200 4700 6200 4750
+Wire Wire Line
+	6100 4700 6100 4750
+Connection ~ 6100 4750
+Wire Wire Line
+	6100 4750 6200 4750
+Wire Wire Line
 	6000 4700 6000 4750
 Connection ~ 6000 4750
+Wire Wire Line
+	6000 4750 6100 4750
 Wire Wire Line
 	5300 4400 5250 4400
@@
 P 5650 5100
 AR Path="/5E6B3291" Ref="C?"  Part="1"
-AR Path="/5E6B2FC0/5E6B3291" Ref="C11"  Part="1"
-F 0 "C11" V 5600 4950 50  0000 C CNN
+AR Path="/5E6B2FC0/5E6B3291" Ref="C19"  Part="1"
+F 0 "C19" V 5600 4950 50  0000 C CNN
 F 1 "100nF" V 5700 4950 50  0000 C CNN
 F 2 "Capacitor_SMD:C_0603_1608Metric" H 5688 4950 50  0001 C CNN
@@
 P 4950 4450
 AR Path="/5E6B329F" Ref="R?"  Part="1"
-AR Path="/5E6B2FC0/5E6B329F" Ref="R13"  Part="1"
-F 0 "R13" V 4900 4250 50  0000 C CNN
+AR Path="/5E6B2FC0/5E6B329F" Ref="R11"  Part="1"
+F 0 "R11" V 4900 4250 50  0000 C CNN
 F 1 "10k" V 5000 4250 50  0000 C CNN
 F 2 "Resistor_SMD:R_0603_1608Metric" V 4880 4450 50  0001 C CNN
@@
 P 4950 4050
 AR Path="/5E6B32AB" Ref="R?"  Part="1"
-AR Path="/5E6B2FC0/5E6B32AB" Ref="R12"  Part="1"
-F 0 "R12" V 4900 3850 50  0000 C CNN
+AR Path="/5E6B2FC0/5E6B32AB" Ref="R10"  Part="1"
+F 0 "R10" V 4900 3850 50  0000 C CNN
 F 1 "10k" V 5000 3850 50  0000 C CNN
 F 2 "Resistor_SMD:R_0603_1608Metric" V 4880 4050 50  0001 C CNN
@@
 P 4900 3850
 AR Path="/5E6B32B7" Ref="R?"  Part="1"
-AR Path="/5E6B2FC0/5E6B32B7" Ref="R11"  Part="1"
-F 0 "R11" V 4850 4050 50  0000 C CNN
+AR Path="/5E6B2FC0/5E6B32B7" Ref="R9"  Part="1"
+F 0 "R9" V 4850 4050 50  0000 C CNN
 F 1 "10k" V 4950 4050 50  0000 C CNN
 F 2 "Resistor_SMD:R_0603_1608Metric" V 4830 3850 50  0001 C CNN
@@
 P 4900 3400
 AR Path="/5E6B32C1" Ref="R?"  Part="1"
-AR Path="/5E6B2FC0/5E6B32C1" Ref="R10"  Part="1"
-F 0 "R10" V 4850 3200 50  0000 C CNN
+AR Path="/5E6B2FC0/5E6B32C1" Ref="R8"  Part="1"
+F 0 "R8" V 4850 3200 50  0000 C CNN
 F 1 "10k" V 4950 3200 50  0000 C CNN
 F 2 "Resistor_SMD:R_0603_1608Metric" V 4830 3400 50  0001 C CNN
@@
 P 4900 4750
 AR Path="/5E6B32CC" Ref="C?"  Part="1"
-AR Path="/5E6B2FC0/5E6B32CC" Ref="C9"  Part="1"
-F 0 "C9" V 4850 4900 50  0000 C CNN
+AR Path="/5E6B2FC0/5E6B32CC" Ref="C17"  Part="1"
+F 0 "C17" V 4850 4900 50  0000 C CNN
 F 1 "6.8nF" V 4950 4900 50  0000 C CNN
 F 2 "Capacitor_SMD:C_0603_1608Metric" H 4938 4600 50  0001 C CNN
@@
 P 4900 4950
 AR Path="/5E6B32D3" Ref="C?"  Part="1"
-AR Path="/5E6B2FC0/5E6B32D3" Ref="C10"  Part="1"
-F 0 "C10" V 4850 4800 50  0000 C CNN
+AR Path="/5E6B2FC0/5E6B32D3" Ref="C18"  Part="1"
+F 0 "C18" V 4850 4800 50  0000 C CNN
 F 1 "120nF" V 4950 4750 50  0000 C CNN
 F 2 "Capacitor_SMD:C_0603_1608Metric" H 4938 4800 50  0001 C CNN
@@
 P 5400 5000
 AR Path="/5E6B32E9" Ref="#PWR?"  Part="1"
-AR Path="/5E6B2FC0/5E6B32E9" Ref="#PWR047"  Part="1"
-F 0 "#PWR047" H 5400 4850 50  0001 C CNN
+AR Path="/5E6B2FC0/5E6B32E9" Ref="#PWR02"  Part="1"
+F 0 "#PWR02" H 5400 4850 50  0001 C CNN
 F 1 "+3.3V" H 5400 5150 50  0000 C CNN
 F 2 "" H 5400 5000 50  0001 C CNN
@@
 P 5350 3250
 AR Path="/5E6B32F9" Ref="#PWR?"  Part="1"
-AR Path="/5E6B2FC0/5E6B32F9" Ref="#PWR046"  Part="1"
-F 0 "#PWR046" H 5350 3100 50  0001 C CNN
+AR Path="/5E6B2FC0/5E6B32F9" Ref="#PWR01"  Part="1"
+F 0 "#PWR01" H 5350 3100 50  0001 C CNN
 F 1 "+3.3V" H 5350 3400 50  0000 C CNN
 F 2 "" H 5350 3250 50  0001 C CNN
@@
 Wire Wire Line
 	5100 4450 5200 4450
+Wire Wire Line
+	6200 4750 6900 4750
+Connection ~ 6200 4750
 Wire Wire Line
 	6600 4500 6500 4500
@@
 Text Notes 7300 6900 0    118  ~ 0
 BNO055 Hierarchical Block (I2C)
-Wire Wire Line
-	6000 4750 6900 4750
-NoConn ~ 7350 4700
 $EndSCHEMATC

Commit message: Fixed broken symbols
Connections:
- wire segments 60 -> 56
Changed lines of the file:
@@
 	5800 4750 5800 4700
-Wire Wire Line
-	6200 4700 6200 4750
-Wire Wire Line
-	6100 4700 6100 4750
-Connection ~ 6100 4750
-Wire Wire Line
-	6100 4750 6200 4750
 Wire Wire Line
 	6000 4700 6000 4750
 Connection ~ 6000 4750
-Wire Wire Line
-	6000 4750 6100 4750
 Wire Wire Line
 	5300 4400 5250 4400
@@
 Wire Wire Line
 	5100 4450 5200 4450
-Wire Wire Line
-	6200 4750 6900 4750
-Connection ~ 6200 4750
 Wire Wire Line
 	6600 4500 6500 4500
@@
 Text Notes 7300 6900 0    118  ~ 0
 BNO055 Hierarchical Block (I2C)
+Wire Wire Line
+	6000 4750 6900 4750
 $EndSCHEMATC

Commit message: Remove duplicated pullup
Parts:
- removed R10, R11: 10k, Resistor_SMD:R_0603_1608Metric, symbol Device:R
Connections:
- wire segments 56 -> 42
Other:
- moved on the sheet: R9
Changed lines of the file:
@@
-$Comp
-L Device:R R?
-U 1 1 5E6B329F
-P 4950 4450
-AR Path="/5E6B329F" Ref="R?"  Part="1"
-AR Path="/5E6B2FC0/5E6B329F" Ref="R11"  Part="1"
-F 0 "R11" V 4900 4250 50  0000 C CNN
-F 1 "10k" V 5000 4250 50  0000 C CNN
-F 2 "Resistor_SMD:R_0603_1608Metric" V 4880 4450 50  0001 C CNN
-F 3 "~" H 4950 4450 50  0001 C CNN
-	1    4950 4450
-	0    1    1    0
-$EndComp
-Wire Wire Line
-	5150 4300 5200 4300
-Wire Wire Line
-	5200 4300 5200 4450
-Connection ~ 5200 4300
-Wire Wire Line
-	5200 4300 5300 4300
-$Comp
-L Device:R R?
-U 1 1 5E6B32AB
-P 4950 4050
-AR Path="/5E6B32AB" Ref="R?"  Part="1"
-AR Path="/5E6B2FC0/5E6B32AB" Ref="R10"  Part="1"
-F 0 "R10" V 4900 3850 50  0000 C CNN
-F 1 "10k" V 5000 3850 50  0000 C CNN
-F 2 "Resistor_SMD:R_0603_1608Metric" V 4880 4050 50  0001 C CNN
-F 3 "~" H 4950 4050 50  0001 C CNN
-	1    4950 4050
-	0    1    1    0
-$EndComp
-Wire Wire Line
-	5150 4200 5200 4200
-Wire Wire Line
-	5200 4200 5200 4050
-Wire Wire Line
-	5200 4200 5300 4200
 $Comp
 L Device:R R?
 U 1 1 5E6B32B7
-P 4900 3850
+P 4900 3900
 AR Path="/5E6B32B7" Ref="R?"  Part="1"
 AR Path="/5E6B2FC0/5E6B32B7" Ref="R9"  Part="1"
-F 0 "R9" V 4850 4050 50  0000 C CNN
-F 1 "10k" V 4950 4050 50  0000 C CNN
-F 2 "Resistor_SMD:R_0603_1608Metric" V 4830 3850 50  0001 C CNN
-F 3 "~" H 4900 3850 50  0001 C CNN
-	1    4900 3850
+F 0 "R9" V 4850 4100 50  0000 C CNN
+F 1 "10k" V 4950 4100 50  0000 C CNN
+F 2 "Resistor_SMD:R_0603_1608Metric" V 4830 3900 50  0001 C CNN
+F 3 "~" H 4900 3900 50  0001 C CNN
+	1    4900 3900
 	0    1    1    0
 $EndComp
@@
 	5050 4750 5250 4750
 Wire Wire Line
-	4650 4050 4650 4250
-Connection ~ 4650 4250
-Wire Wire Line
-	4650 4250 4650 4450
-Wire Wire Line
 	5200 3550 5300 3550
 Wire Wire Line
@@
 Wire Wire Line
 	5500 5100 5400 5100
-Wire Wire Line
-	5300 3900 5200 3900
-Wire Wire Line
-	5200 3900 5200 3850
-Wire Wire Line
-	5200 3850 5050 3850
 Wire Wire Line
 	6000 3250 6000 3300
@@
 	4550 3400 4550 3250
 Wire Wire Line
-	4750 3850 4550 3850
-Connection ~ 4550 3850
-Wire Wire Line
-	4550 3850 4550 3400
-Connection ~ 4550 4250
-Wire Wire Line
-	4550 4250 4550 3850
+	4750 3900 4550 3900
 Wire Wire Line
 	4750 4750 4550 4750
 Connection ~ 4550 4750
 Wire Wire Line
-	4550 4750 4550 4250
-Wire Wire Line
 	5400 5100 5400 5000
 Wire Wire Line
 	5800 4750 5800 5100
-Wire Wire Line
-	4550 4250 4650 4250
-Wire Wire Line
-	4800 4450 4650 4450
-Wire Wire Line
-	4650 4050 4800 4050
-Wire Wire Line
-	5100 4050 5200 4050
-Wire Wire Line
-	5100 4450 5200 4450
 Wire Wire Line
 	6600 4500 6500 4500
@@
 Text HLabel 5150 4300 0    50   Output ~ 0
 SCL
-Connection ~ 5200 4200
 Text Notes 7300 6900 0    118  ~ 0
 BNO055 Hierarchical Block (I2C)
 Wire Wire Line
 	6000 4750 6900 4750
+Wire Wire Line
+	5150 4300 5300 4300
+Wire Wire Line
+	5150 4200 5300 4200
+Connection ~ 4550 3900
+Wire Wire Line
+	4550 3900 4550 4750
+Wire Wire Line
+	4550 3400 4550 3900
+Wire Wire Line
+	5050 3900 5300 3900
 $EndSCHEMATC

Commit message: add symbol libraries, and cleanup
Parts:
- C1201: renamed from C20; DIGIKEY (none) -> 399-1100-1-ND; MANF (none) -> C0603C104Z3VACTU
- C1202: renamed from C17; DIGIKEY (none) -> 1292-1459-1-ND; MANF (none) -> 0603B682K500CT
- C1203: renamed from C18; DIGIKEY (none) -> 311-4056-1-ND; MANF (none) -> CC0603KRX7R6BB124
- C1204: renamed from C19; DIGIKEY (none) -> 399-1100-1-ND; MANF (none) -> C0603C104Z3VACTU
- R1201: renamed from R9; DIGIKEY (none) -> 311-10KGRCT-ND; MANF (none) -> RC0603JR-0710KL
- R1202: renamed from R8; DIGIKEY (none) -> 311-10KGRCT-ND; MANF (none) -> RC0603JR-0710KL
- U1201: renamed from U4; DIGIKEY (none) -> 828-1058-1-ND; MANF (none) -> BNO055
Connections:
- wire segments 42 -> 36
Other:
- moved on the sheet: C1202, C1203, C1204, R1201, R1202
