File: BNO055/BNO055.sch (KiCad schematic (older format))
At the start: 7 parts, among them U1201 BNO055

Commit message: fix BNO055 schematic
Parts:
- removed C1202: 6.8nF, Capacitor_SMD:C_0603_1608Metric, symbol Device:C
- C1201: value 100nF -> 1uF; DIGIKEY 399-1100-1-ND -> 1276-1182-1-ND; MANF C0603C104Z3VACTU -> CL10A105KP8NNNC
- renumbered C1203 to C1202, C1204 to C1203
Connections:
- wire segments 36 -> 34
Changed lines of the file:
@@
 P 6750 4500
 F 0 "C1201" V 6900 4500 50  0000 C CNN
-F 1 "100nF" V 7000 4500 50  0000 C CNN
+F 1 "1uF" V 7000 4500 50  0000 C CNN
 F 2 "Capacitor_SMD:C_0603_1608Metric" H 6788 4350 50  0001 C CNN
 F 3 "~" H 6750 4500 50  0001 C CNN
-F 4 "C0603C104Z3VACTU" H 6750 4500 50  0001 C CNN "MANF"
-F 5 "399-1100-1-ND" H 6750 4500 50  0001 C CNN "DIGIKEY"
+F 4 "CL10A105KP8NNNC" H 6750 4500 50  0001 C CNN "MANF"
+F 5 "1276-1182-1-ND" H 6750 4500 50  0001 C CNN "DIGIKEY"
 	1    6750 4500
 	0    1    1    0
@@
 $Comp
 L Device:C C1202
-U 1 1 5E6B32CC
-P 8100 3600
-F 0 "C1202" V 8250 3600 50  0000 C CNN
-F 1 "6.8nF" V 8350 3600 50  0000 C CNN
-F 2 "Capacitor_SMD:C_0603_1608Metric" H 8138 3450 50  0001 C CNN
-F 3 "~" H 8100 3600 50  0001 C CNN
-F 4 "1292-1459-1-ND" H 8100 3600 50  0001 C CNN "DIGIKEY"
-F 5 "0603B682K500CT" H 8100 3600 50  0001 C CNN "MANF"
-	1    8100 3600
-	0    1    1    0
-$EndComp
-$Comp
-L Device:C C1203
 U 1 1 5E6B32D3
 P 8100 4000
-F 0 "C1203" V 8250 4000 50  0000 C CNN
+F 0 "C1202" V 8250 4000 50  0000 C CNN
 F 1 "120nF" V 8350 4000 50  0000 C CNN
 F 2 "Capacitor_SMD:C_0603_1608Metric" H 8138 3850 50  0001 C CNN
@@
 L power:+3.3V #PWR01207
 U 1 1 5E6B32E9
-P 7950 3400
-F 0 "#PWR01207" H 7950 3250 50  0001 C CNN
-F 1 "+3.3V" H 7950 3550 50  0000 C CNN
-F 2 "" H 7950 3400 50  0001 C CNN
-F 3 "" H 7950 3400 50  0001 C CNN
-	1    7950 3400
+P 7950 3750
+F 0 "#PWR01207" H 7950 3600 50  0001 C CNN
+F 1 "+3.3V" H 7950 3900 50  0000 C CNN
+F 2 "" H 7950 3750 50  0001 C CNN
+F 3 "" H 7950 3750 50  0001 C CNN
+	1    7950 3750
 	1    0    0    -1
 $EndComp
@@
 	5150 4300 5300 4300
 $Comp
-L Device:C C1204
+L Device:C C1203
 U 1 1 5E6B3291
 P 8100 4400
-F 0 "C1204" V 8250 4400 50  0000 C CNN
+F 0 "C1203" V 8250 4400 50  0000 C CNN
 F 1 "100nF" V 8350 4400 50  0000 C CNN
 F 2 "Capacitor_SMD:C_0603_1608Metric" H 8138 4250 50  0001 C CNN
@@
 L power:GND #PWR01208
 U 1 1 5F9BE479
-P 8450 3400
-F 0 "#PWR01208" H 8450 3150 50  0001 C CNN
-F 1 "GND" H 8455 3227 50  0000 C CNN
-F 2 "" H 8450 3400 50  0001 C CNN
-F 3 "" H 8450 3400 50  0001 C CNN
-	1    8450 3400
-	1    0    0    -1
-$EndComp
-Wire Wire Line
-	8450 3400 8250 3400
-Wire Wire Line
-	8250 3400 8250 3600
-Connection ~ 8250 3600
-Wire Wire Line
-	8250 3600 8250 4000
-Connection ~ 8250 4000
+P 8450 3750
+F 0 "#PWR01208" H 8450 3500 50  0001 C CNN
+F 1 "GND" H 8455 3577 50  0000 C CNN
+F 2 "" H 8450 3750 50  0001 C CNN
+F 3 "" H 8450 3750 50  0001 C CNN
+	1    8450 3750
+	1    0    0    -1
+$EndComp
+Wire Wire Line
+	8450 3750 8250 3750
 Wire Wire Line
 	8250 4000 8250 4400
 Wire Wire Line
 	7950 4400 7950 4000
-Connection ~ 7950 3600
-Wire Wire Line
-	7950 3600 7950 3400
-Connection ~ 7950 4000
-Wire Wire Line
-	7950 4000 7950 3600
 $Comp
 L power:GND #PWR01203
@@
 Wire Wire Line
 	7150 4400 6900 4400
+Wire Wire Line
+	7950 4000 7950 3750
+Connection ~ 7950 4000
+Wire Wire Line
+	8250 4000 8250 3750
+Connection ~ 8250 4000
 $EndSCHEMATC
