File: STM32F401RET6/STM32F401RET6.sch (KiCad schematic (older format))
At the start: 12 parts

Commit message: Update Schematic blocks
Parts:
- gave numbers to parts that had none: 12
Changed lines of the file:
@@
 $Descr A4 11693 8268
 encoding utf-8
-Sheet 4 5
+Sheet 4 6
 Title ""
 Date ""
@@
 $EndDescr
 $Comp
-L MCU_ST_STM32F4:STM32F401RETx U?
+L MCU_ST_STM32F4:STM32F401RETx U4
 U 1 1 5DE1731E
 P 5250 4100
-F 0 "U?" H 5800 5950 50  0000 C CNN
+F 0 "U4" H 5800 5950 50  0000 C CNN
 F 1 "STM32F401RETx" H 5800 5850 50  0000 C CNN
 F 2 "Package_QFP:LQFP-64_10x10mm_P0.5mm" H 4650 2400 50  0001 R CNN
@@
 	5250 2300 5250 2400
 $Comp
-L power:GND #PWR?
+L power:GND #PWR063
 U 1 1 5DE18883
 P 5250 6000
-F 0 "#PWR?" H 5250 5750 50  0001 C CNN
+F 0 "#PWR063" H 5250 5750 50  0001 C CNN
 F 1 "GND" H 5255 5827 50  0000 C CNN
 F 2 "" H 5250 6000 50  0001 C CNN
@@
 	5250 6000 5250 5900
 $Comp
-L Device:C C?
+L Device:C C16
 U 1 1 5DE19367
 P 8650 3750
-F 0 "C?" H 8765 3796 50  0000 L CNN
+F 0 "C16" H 8765 3796 50  0000 L CNN
 F 1 "0.1uF" H 8765 3705 50  0000 L CNN
 F 2 "" H 8688 3600 50  0001 C CNN
@@
 $EndComp
 $Comp
-L Device:C C?
+L Device:C C18
 U 1 1 5DE19787
 P 9100 3750
-F 0 "C?" H 9215 3796 50  0000 L CNN
+F 0 "C18" H 9215 3796 50  0000 L CNN
 F 1 "0.1uF" H 9215 3705 50  0000 L CNN
 F 2 "" H 9138 3600 50  0001 C CNN
@@
 $EndComp
 $Comp
-L Device:C C?
+L Device:C C19
 U 1 1 5DE19D37
 P 9550 3750
-F 0 "C?" H 9665 3796 50  0000 L CNN
+F 0 "C19" H 9665 3796 50  0000 L CNN
 F 1 "0.1uF" H 9665 3705 50  0000 L CNN
 F 2 "" H 9588 3600 50  0001 C CNN
@@
 $EndComp
 $Comp
-L Device:C C?
+L Device:C C20
 U 1 1 5DE19F0D
 P 10000 3750
-F 0 "C?" H 10115 3796 50  0000 L CNN
+F 0 "C20" H 10115 3796 50  0000 L CNN
 F 1 "0.1uF" H 10115 3705 50  0000 L CNN
 F 2 "" H 10038 3600 50  0001 C CNN
@@
 	8200 3900 8650 3900
 $Comp
-L Device:C C?
+L Device:C C13
 U 1 1 5DE19136
 P 8200 3750
-F 0 "C?" H 8315 3796 50  0000 L CNN
+F 0 "C13" H 8315 3796 50  0000 L CNN
 F 1 "10uF" H 8315 3705 50  0000 L CNN
 F 2 "" H 8238 3600 50  0001 C CNN
@@
 $EndComp
 $Comp
-L power:GND #PWR?
+L power:GND #PWR065
 U 1 1 5DE18B06
 P 8000 3900
-F 0 "#PWR?" H 8000 3650 50  0001 C CNN
+F 0 "#PWR065" H 8000 3650 50  0001 C CNN
 F 1 "GND" H 8005 3727 50  0000 C CNN
 F 2 "" H 8000 3900 50  0001 C CNN
@@
 $EndComp
 $Comp
-L power:GND #PWR?
+L power:GND #PWR067
 U 1 1 5DE1D921
 P 8000 4650
-F 0 "#PWR?" H 8000 4400 50  0001 C CNN
+F 0 "#PWR067" H 8000 4400 50  0001 C CNN
 F 1 "GND" H 8005 4477 50  0000 C CNN
 F 2 "" H 8000 4650 50  0001 C CNN
@@
 $EndComp
 $Comp
-L Device:C C?
+L Device:C C14
 U 1 1 5DE1DB7A
 P 8250 4500
-F 0 "C?" H 8365 4546 50  0000 L CNN
+F 0 "C14" H 8365 4546 50  0000 L CNN
 F 1 "0.1uF" H 8365 4455 50  0000 L CNN
 F 2 "" H 8288 4350 50  0001 C CNN
@@
 	8250 4350 8000 4350
 $Comp
-L Device:C C?
+L Device:C C15
 U 1 1 5DE1EBB5
 P 8250 5250
-F 0 "C?" H 8365 5296 50  0000 L CNN
+F 0 "C15" H 8365 5296 50  0000 L CNN
 F 1 "0.1uF" H 8365 5205 50  0000 L CNN
 F 2 "" H 8288 5100 50  0001 C CNN
@@
 $EndComp
 $Comp
-L power:GND #PWR?
+L power:GND #PWR069
 U 1 1 5DE1F4FA
 P 8000 5400
-F 0 "#PWR?" H 8000 5150 50  0001 C CNN
+F 0 "#PWR069" H 8000 5150 50  0001 C CNN
 F 1 "GND" H 8005 5227 50  0000 C CNN
 F 2 "" H 8000 5400 50  0001 C CNN
@@
 $EndComp
 $Comp
-L Device:C C?
+L Device:C C17
 U 1 1 5DE17F46
 P 8700 5250
-F 0 "C?" H 8815 5296 50  0000 L CNN
+F 0 "C17" H 8815 5296 50  0000 L CNN
 F 1 "1uF" H 8815 5205 50  0000 L CNN
 F 2 "" H 8738 5100 50  0001 C CNN
@@
 VDD decoupling caps
 $Comp
-L Device:C C?
+L Device:C C12
 U 1 1 5DE1ABC6
 P 3950 3150
-F 0 "C?" H 4065 3196 50  0000 L CNN
+F 0 "C12" H 4065 3196 50  0000 L CNN
 F 1 "4.7uF" H 4065 3105 50  0000 L CNN
 F 2 "" H 3988 3000 50  0001 C CNN
@@
 $EndComp
 $Comp
-L power:GND #PWR?
+L power:GND #PWR060
 U 1 1 5DE1B283
 P 3950 3300
-F 0 "#PWR?" H 3950 3050 50  0001 C CNN
+F 0 "#PWR060" H 3950 3050 50  0001 C CNN
 F 1 "GND" H 3955 3127 50  0000 C CNN
 F 2 "" H 3950 3300 50  0001 C CNN
@@
 	3950 3000 4300 3000
 $Comp
-L Device:C C?
+L Device:C C11
 U 1 1 5DE1BE22
 P 3150 2750
-F 0 "C?" H 3265 2796 50  0000 L CNN
+F 0 "C11" H 3265 2796 50  0000 L CNN
 F 1 "0.1uF" H 3265 2705 50  0000 L CNN
 F 2 "" H 3188 2600 50  0001 C CNN
@@
 	2950 2600 3150 2600
 $Comp
-L power:GND #PWR?
+L power:GND #PWR058
 U 1 1 5DE1D367
 P 3150 2900
-F 0 "#PWR?" H 3150 2650 50  0001 C CNN
+F 0 "#PWR058" H 3150 2650 50  0001 C CNN
 F 1 "GND" H 3155 2727 50  0000 C CNN
 F 2 "" H 3150 2900 50  0001 C CNN
@@
 Connection ~ 3150 2600
 $Comp
-L Device:R R?
+L Device:R R8
 U 1 1 5DE1E2D2
 P 3600 2950
-F 0 "R?" H 3670 2996 50  0000 L CNN
+F 0 "R8" H 3670 2996 50  0000 L CNN
 F 1 "10K" H 3670 2905 50  0000 L CNN
 F 2 "" V 3530 2950 50  0001 C CNN
@@
 $EndComp
 $Comp
-L power:GND #PWR?
+L power:GND #PWR059
 U 1 1 5DE1E857
 P 3600 3100
-F 0 "#PWR?" H 3600 2850 50  0001 C CNN
+F 0 "#PWR059" H 3600 2850 50  0001 C CNN
 F 1 "GND" H 3605 2927 50  0000 C CNN
 F 2 "" H 3600 3100 50  0001 C CNN
@@
 SPI2 nSS / I2S2 WS, I2C1 SDA, SDIO D5
 $Comp
-L power:+3.3V #PWR?
+L power:+3.3V #PWR062
 U 1 1 5DE1F0DC
 P 5250 2300
-F 0 "#PWR?" H 5250 2150 50  0001 C CNN
+F 0 "#PWR062" H 5250 2150 50  0001 C CNN
 F 1 "+3.3V" H 5265 2473 50  0000 C CNN
 F 2 "" H 5250 2300 50  0001 C CNN
@@
 $EndComp
 $Comp
-L power:+3.3V #PWR?
+L power:+3.3V #PWR064
 U 1 1 5DE22E45
 P 8000 3600
-F 0 "#PWR?" H 8000 3450 50  0001 C CNN
+F 0 "#PWR064" H 8000 3450 50  0001 C CNN
 F 1 "+3.3V" H 8015 3773 50  0000 C CNN
 F 2 "" H 8000 3600 50  0001 C CNN
@@
 $EndComp
 $Comp
-L power:+3.3V #PWR?
+L power:+3.3V #PWR066
 U 1 1 5DE235AC
 P 8000 4350
-F 0 "#PWR?" H 8000 4200 50  0001 C CNN
+F 0 "#PWR066" H 8000 4200 50  0001 C CNN
 F 1 "+3.3V" H 8015 4523 50  0000 C CNN
 F 2 "" H 8000 4350 50  0001 C CNN
@@
 $EndComp
 $Comp
-L power:+3.3V #PWR?
+L power:+3.3V #PWR068
 U 1 1 5DE2397A
 P 8000 5100
-F 0 "#PWR?" H 8000 4950 50  0001 C CNN
+F 0 "#PWR068" H 8000 4950 50  0001 C CNN
 F 1 "+3.3V" H 8015 5273 50  0000 C CNN
 F 2 "" H 8000 5100 50  0001 C CNN
@@
 STM32F401RET6 Hierarchical Block
 $Comp
-L power:+3.3V #PWR?
+L power:+3.3V #PWR061
 U 1 1 5DE2F79B
 P 4550 3150
-F 0 "#PWR?" H 4550 3000 50  0001 C CNN
+F 0 "#PWR061" H 4550 3000 50  0001 C CNN
 F 1 "+3.3V" H 4565 3323 50  0000 C CNN
 F 2 "" H 4550 3150 50  0001 C CNN
@@
 	4550 3100 4550 3150
 $Comp
-L power:PWR_FLAG #FLG?
+L power:PWR_FLAG #FLG05
 U 1 1 5DE3436C
 P 4300 3300
-F 0 "#FLG?" H 4300 3375 50  0001 C CNN
+F 0 "#FLG05" H 4300 3375 50  0001 C CNN
 F 1 "PWR_FLAG" H 4300 3473 50  0000 C CNN
 F 2 "" H 4300 3300 50  0001 C CNN

Commit message: Update schematics
Parts:
- renumbered C11 to C16, C12 to C17, C13 to C18, C14 to C19, C15 to C20, C16 to C21, C17 to C22, C18 to C23, C19 to C24, C20 to C25, R8 to R18, U4 to U7
Changed lines of the file:
@@
 $Descr A4 11693 8268
 encoding utf-8
-Sheet 4 6
+Sheet 6 6
 Title ""
 Date ""
@@
 $EndDescr
 $Comp
-L MCU_ST_STM32F4:STM32F401RETx U4
+L MCU_ST_STM32F4:STM32F401RETx U7
 U 1 1 5DE1731E
 P 5250 4100
-F 0 "U4" H 5800 5950 50  0000 C CNN
+F 0 "U7" H 5800 5950 50  0000 C CNN
 F 1 "STM32F401RETx" H 5800 5850 50  0000 C CNN
 F 2 "Package_QFP:LQFP-64_10x10mm_P0.5mm" H 4650 2400 50  0001 R CNN
@@
 	5250 2300 5250 2400
 $Comp
-L power:GND #PWR063
+L power:GND #PWR093
 U 1 1 5DE18883
 P 5250 6000
-F 0 "#PWR063" H 5250 5750 50  0001 C CNN
+F 0 "#PWR093" H 5250 5750 50  0001 C CNN
 F 1 "GND" H 5255 5827 50  0000 C CNN
 F 2 "" H 5250 6000 50  0001 C CNN
@@
 	5250 6000 5250 5900
 $Comp
-L Device:C C16
+L Device:C C21
 U 1 1 5DE19367
 P 8650 3750
-F 0 "C16" H 8765 3796 50  0000 L CNN
+F 0 "C21" H 8765 3796 50  0000 L CNN
 F 1 "0.1uF" H 8765 3705 50  0000 L CNN
 F 2 "" H 8688 3600 50  0001 C CNN
@@
 $EndComp
 $Comp
-L Device:C C18
+L Device:C C23
 U 1 1 5DE19787
 P 9100 3750
-F 0 "C18" H 9215 3796 50  0000 L CNN
+F 0 "C23" H 9215 3796 50  0000 L CNN
 F 1 "0.1uF" H 9215 3705 50  0000 L CNN
 F 2 "" H 9138 3600 50  0001 C CNN
@@
 $EndComp
 $Comp
-L Device:C C19
+L Device:C C24
 U 1 1 5DE19D37
 P 9550 3750
-F 0 "C19" H 9665 3796 50  0000 L CNN
+F 0 "C24" H 9665 3796 50  0000 L CNN
 F 1 "0.1uF" H 9665 3705 50  0000 L CNN
 F 2 "" H 9588 3600 50  0001 C CNN
@@
 $EndComp
 $Comp
-L Device:C C20
+L Device:C C25
 U 1 1 5DE19F0D
 P 10000 3750
-F 0 "C20" H 10115 3796 50  0000 L CNN
+F 0 "C25" H 10115 3796 50  0000 L CNN
 F 1 "0.1uF" H 10115 3705 50  0000 L CNN
 F 2 "" H 10038 3600 50  0001 C CNN
@@
 	8200 3900 8650 3900
 $Comp
-L Device:C C13
+L Device:C C18
 U 1 1 5DE19136
 P 8200 3750
-F 0 "C13" H 8315 3796 50  0000 L CNN
+F 0 "C18" H 8315 3796 50  0000 L CNN
 F 1 "10uF" H 8315 3705 50  0000 L CNN
 F 2 "" H 8238 3600 50  0001 C CNN
@@
 $EndComp
 $Comp
-L power:GND #PWR065
+L power:GND #PWR095
 U 1 1 5DE18B06
 P 8000 3900
-F 0 "#PWR065" H 8000 3650 50  0001 C CNN
+F 0 "#PWR095" H 8000 3650 50  0001 C CNN
 F 1 "GND" H 8005 3727 50  0000 C CNN
 F 2 "" H 8000 3900 50  0001 C CNN
@@
 $EndComp
 $Comp
-L power:GND #PWR067
+L power:GND #PWR097
 U 1 1 5DE1D921
 P 8000 4650
-F 0 "#PWR067" H 8000 4400 50  0001 C CNN
+F 0 "#PWR097" H 8000 4400 50  0001 C CNN
 F 1 "GND" H 8005 4477 50  0000 C CNN
 F 2 "" H 8000 4650 50  0001 C CNN
@@
 $EndComp
 $Comp
-L Device:C C14
+L Device:C C19
 U 1 1 5DE1DB7A
 P 8250 4500
-F 0 "C14" H 8365 4546 50  0000 L CNN
+F 0 "C19" H 8365 4546 50  0000 L CNN
 F 1 "0.1uF" H 8365 4455 50  0000 L CNN
 F 2 "" H 8288 4350 50  0001 C CNN
@@
 	8250 4350 8000 4350
 $Comp
-L Device:C C15
+L Device:C C20
 U 1 1 5DE1EBB5
 P 8250 5250
-F 0 "C15" H 8365 5296 50  0000 L CNN
+F 0 "C20" H 8365 5296 50  0000 L CNN
 F 1 "0.1uF" H 8365 5205 50  0000 L CNN
 F 2 "" H 8288 5100 50  0001 C CNN
@@
 $EndComp
 $Comp
-L power:GND #PWR069
+L power:GND #PWR099
 U 1 1 5DE1F4FA
 P 8000 5400
-F 0 "#PWR069" H 8000 5150 50  0001 C CNN
+F 0 "#PWR099" H 8000 5150 50  0001 C CNN
 F 1 "GND" H 8005 5227 50  0000 C CNN
 F 2 "" H 8000 5400 50  0001 C CNN
@@
 $EndComp
 $Comp
-L Device:C C17
+L Device:C C22
 U 1 1 5DE17F46
 P 8700 5250
-F 0 "C17" H 8815 5296 50  0000 L CNN
+F 0 "C22" H 8815 5296 50  0000 L CNN
 F 1 "1uF" H 8815 5205 50  0000 L CNN
 F 2 "" H 8738 5100 50  0001 C CNN
@@
 VDD decoupling caps
 $Comp
-L Device:C C12
+L Device:C C17
 U 1 1 5DE1ABC6
 P 3950 3150
-F 0 "C12" H 4065 3196 50  0000 L CNN
+F 0 "C17" H 4065 3196 50  0000 L CNN
 F 1 "4.7uF" H 4065 3105 50  0000 L CNN
 F 2 "" H 3988 3000 50  0001 C CNN
@@
 $EndComp
 $Comp
-L power:GND #PWR060
+L power:GND #PWR090
 U 1 1 5DE1B283
 P 3950 3300
-F 0 "#PWR060" H 3950 3050 50  0001 C CNN
+F 0 "#PWR090" H 3950 3050 50  0001 C CNN
 F 1 "GND" H 3955 3127 50  0000 C CNN
 F 2 "" H 3950 3300 50  0001 C CNN
@@
 	3950 3000 4300 3000
 $Comp
-L Device:C C11
+L Device:C C16
 U 1 1 5DE1BE22
 P 3150 2750
-F 0 "C11" H 3265 2796 50  0000 L CNN
+F 0 "C16" H 3265 2796 50  0000 L CNN
 F 1 "0.1uF" H 3265 2705 50  0000 L CNN
 F 2 "" H 3188 2600 50  0001 C CNN
@@
 	2950 2600 3150 2600
 $Comp
-L power:GND #PWR058
+L power:GND #PWR088
 U 1 1 5DE1D367
 P 3150 2900
-F 0 "#PWR058" H 3150 2650 50  0001 C CNN
+F 0 "#PWR088" H 3150 2650 50  0001 C CNN
 F 1 "GND" H 3155 2727 50  0000 C CNN
 F 2 "" H 3150 2900 50  0001 C CNN
@@
 Connection ~ 3150 2600
 $Comp
-L Device:R R8
+L Device:R R18
 U 1 1 5DE1E2D2
 P 3600 2950
-F 0 "R8" H 3670 2996 50  0000 L CNN
+F 0 "R18" H 3670 2996 50  0000 L CNN
 F 1 "10K" H 3670 2905 50  0000 L CNN
 F 2 "" V 3530 2950 50  0001 C CNN
@@
 $EndComp
 $Comp
-L power:GND #PWR059
+L power:GND #PWR089
 U 1 1 5DE1E857
 P 3600 3100
-F 0 "#PWR059" H 3600 2850 50  0001 C CNN
+F 0 "#PWR089" H 3600 2850 50  0001 C CNN
 F 1 "GND" H 3605 2927 50  0000 C CNN
 F 2 "" H 3600 3100 50  0001 C CNN
@@
 SPI2 nSS / I2S2 WS, I2C1 SDA, SDIO D5
 $Comp
-L power:+3.3V #PWR062
+L power:+3.3V #PWR092
 U 1 1 5DE1F0DC
 P 5250 2300
-F 0 "#PWR062" H 5250 2150 50  0001 C CNN
+F 0 "#PWR092" H 5250 2150 50  0001 C CNN
 F 1 "+3.3V" H 5265 2473 50  0000 C CNN
 F 2 "" H 5250 2300 50  0001 C CNN
@@
 $EndComp
 $Comp
-L power:+3.3V #PWR064
+L power:+3.3V #PWR094
 U 1 1 5DE22E45
 P 8000 3600
-F 0 "#PWR064" H 8000 3450 50  0001 C CNN
+F 0 "#PWR094" H 8000 3450 50  0001 C CNN
 F 1 "+3.3V" H 8015 3773 50  0000 C CNN
 F 2 "" H 8000 3600 50  0001 C CNN
@@
 $EndComp
 $Comp
-L power:+3.3V #PWR066
+L power:+3.3V #PWR096
 U 1 1 5DE235AC
 P 8000 4350
-F 0 "#PWR066" H 8000 4200 50  0001 C CNN
+F 0 "#PWR096" H 8000 4200 50  0001 C CNN
 F 1 "+3.3V" H 8015 4523 50  0000 C CNN
 F 2 "" H 8000 4350 50  0001 C CNN
@@
 $EndComp
 $Comp
-L power:+3.3V #PWR068
+L power:+3.3V #PWR098
 U 1 1 5DE2397A
 P 8000 5100
-F 0 "#PWR068" H 8000 4950 50  0001 C CNN
+F 0 "#PWR098" H 8000 4950 50  0001 C CNN
 F 1 "+3.3V" H 8015 5273 50  0000 C CNN
 F 2 "" H 8000 5100 50  0001 C CNN
@@
 STM32F401RET6 Hierarchical Block
 $Comp
-L power:+3.3V #PWR061
+L power:+3.3V #PWR091
 U 1 1 5DE2F79B
 P 4550 3150
-F 0 "#PWR061" H 4550 3000 50  0001 C CNN
+F 0 "#PWR091" H 4550 3000 50  0001 C CNN
 F 1 "+3.3V" H 4565 3323 50  0000 C CNN
 F 2 "" H 4550 3150 50  0001 C CNN
