File: CAS_bus/CAS_bus.sch (KiCad schematic (older format))
At the start: 1 part, among them J1001 CAS_stacking

Commit message: slightly clearer
Parts:
- renumbered J1001 to J5
Changed lines of the file:
@@
 EESchema Schematic File Version 4
-EELAYER 30 0
+LIBS:Prop-cache
+EELAYER 26 0
 EELAYER END
 $Descr A4 11693 8268
 encoding utf-8
-Sheet 2 2
+Sheet 5 8
 Title ""
 Date ""
@@
 SPI0_nSS8
 $Comp
-L power:+5V #PWR02
+L power:+5V #PWR0113
 U 1 1 5EAFC0A6
 P 4300 2000
-F 0 "#PWR02" H 4300 1850 50  0001 C CNN
+F 0 "#PWR0113" H 4300 1850 50  0001 C CNN
 F 1 "+5V" V 4315 2128 50  0000 L CNN
 F 2 "" H 4300 2000 50  0001 C CNN
@@
 $EndComp
 $Comp
-L power:+5V #PWR013
+L power:+5V #PWR0114
 U 1 1 5EAFC439
 P 6000 2000
-F 0 "#PWR013" H 6000 1850 50  0001 C CNN
+F 0 "#PWR0114" H 6000 1850 50  0001 C CNN
 F 1 "+5V" V 6015 2128 50  0000 L CNN
 F 2 "" H 6000 2000 50  0001 C CNN
@@
 $EndComp
 $Comp
-L power:+3.3V #PWR019
+L power:+3.3V #PWR0115
 U 1 1 5EAFC7C9
 P 6000 3500
-F 0 "#PWR019" H 6000 3350 50  0001 C CNN
+F 0 "#PWR0115" H 6000 3350 50  0001 C CNN
 F 1 "+3.3V" V 6015 3628 50  0000 L CNN
 F 2 "" H 6000 3500 50  0001 C CNN
@@
 $EndComp
 $Comp
-L power:+BATT #PWR07
+L power:+BATT #PWR0116
 U 1 1 5EAFCF46
 P 4300 3700
-F 0 "#PWR07" H 4300 3550 50  0001 C CNN
+F 0 "#PWR0116" H 4300 3550 50  0001 C CNN
 F 1 "+BATT" V 4315 3827 50  0000 L CNN
 F 2 "" H 4300 3700 50  0001 C CNN
@@
 $EndComp
 $Comp
-L power:+BATT #PWR021
+L power:+BATT #PWR0117
 U 1 1 5EAFD5BD
 P 6000 3700
-F 0 "#PWR021" H 6000 3550 50  0001 C CNN
+F 0 "#PWR0117" H 6000 3550 50  0001 C CNN
 F 1 "+BATT" V 6015 3828 50  0000 L CNN
 F 2 "" H 6000 3700 50  0001 C CNN
@@
 $EndComp
 $Comp
-L power:GND #PWR015
+L power:GND #PWR0118
 U 1 1 5EAFD991
 P 6000 2500
-F 0 "#PWR015" H 6000 2250 50  0001 C CNN
+F 0 "#PWR0118" H 6000 2250 50  0001 C CNN
 F 1 "GND" V 6005 2372 50  0000 R CNN
 F 2 "" H 6000 2500 50  0001 C CNN
@@
 $EndComp
 $Comp
-L power:GND #PWR04
+L power:GND #PWR0119
 U 1 1 5EAFDD6C
 P 4300 2500
-F 0 "#PWR04" H 4300 2250 50  0001 C CNN
+F 0 "#PWR0119" H 4300 2250 50  0001 C CNN
 F 1 "GND" V 4305 2372 50  0000 R CNN
 F 2 "" H 4300 2500 50  0001 C CNN
@@
 $EndComp
 $Comp
-L power:GND #PWR020
+L power:GND #PWR0120
 U 1 1 5EAFEFF0
 P 6000 3600
-F 0 "#PWR020" H 6000 3350 50  0001 C CNN
+F 0 "#PWR0120" H 6000 3350 50  0001 C CNN
 F 1 "GND" V 6005 3472 50  0000 R CNN
 F 2 "" H 6000 3600 50  0001 C CNN
@@
 	5850 2000 6000 2000
 $Comp
-L power:GND #PWR012
+L power:GND #PWR0121
 U 1 1 5EB0043E
 P 6000 1900
-F 0 "#PWR012" H 6000 1650 50  0001 C CNN
+F 0 "#PWR0121" H 6000 1650 50  0001 C CNN
 F 1 "GND" V 6005 1772 50  0000 R CNN
 F 2 "" H 6000 1900 50  0001 C CNN
@@
 $EndComp
 $Comp
-L power:GND #PWR014
+L power:GND #PWR0122
 U 1 1 5EB00872
 P 6000 2100
-F 0 "#PWR014" H 6000 1850 50  0001 C CNN
+F 0 "#PWR0122" H 6000 1850 50  0001 C CNN
 F 1 "GND" V 6005 1972 50  0000 R CNN
 F 2 "" H 6000 2100 50  0001 C CNN
@@
 $EndComp
 $Comp
-L power:GND #PWR01
+L power:GND #PWR0123
 U 1 1 5EB00CA1
 P 4300 1900
-F 0 "#PWR01" H 4300 1650 50  0001 C CNN
+F 0 "#PWR0123" H 4300 1650 50  0001 C CNN
 F 1 "GND" V 4305 1772 50  0000 R CNN
 F 2 "" H 4300 1900 50  0001 C CNN
@@
 $EndComp
 $Comp
-L power:GND #PWR03
+L power:GND #PWR0124
 U 1 1 5EB01123
 P 4300 2100
-F 0 "#PWR03" H 4300 1850 50  0001 C CNN
+F 0 "#PWR0124" H 4300 1850 50  0001 C CNN
 F 1 "GND" V 4305 1972 50  0000 R CNN
 F 2 "" H 4300 2100 50  0001 C CNN
@@
 SPIHS_nSS2
 $Comp
-L power:GND #PWR08
+L power:GND #PWR0125
 U 1 1 5EB1964E
 P 4300 4200
-F 0 "#PWR08" H 4300 3950 50  0001 C CNN
+F 0 "#PWR0125" H 4300 3950 50  0001 C CNN
 F 1 "GND" V 4305 4072 50  0000 R CNN
 F 2 "" H 4300 4200 50  0001 C CNN
@@
 $EndComp
 $Comp
-L power:GND #PWR09
+L power:GND #PWR0126
 U 1 1 5EB19A77
 P 4300 4300
-F 0 "#PWR09" H 4300 4050 50  0001 C CNN
+F 0 "#PWR0126" H 4300 4050 50  0001 C CNN
 F 1 "GND" V 4305 4172 50  0000 R CNN
 F 2 "" H 4300 4300 50  0001 C CNN
@@
 $EndComp
 $Comp
-L power:GND #PWR010
+L power:GND #PWR0127
 U 1 1 5EB19EAC
 P 4300 4500
-F 0 "#PWR010" H 4300 4250 50  0001 C CNN
+F 0 "#PWR0127" H 4300 4250 50  0001 C CNN
 F 1 "GND" V 4305 4372 50  0000 R CNN
 F 2 "" H 4300 4500 50  0001 C CNN
@@
 $EndComp
 $Comp
-L power:GND #PWR011
+L power:GND #PWR0128
 U 1 1 5EB1A2ED
 P 4300 4700
-F 0 "#PWR011" H 4300 4450 50  0001 C CNN
+F 0 "#PWR0128" H 4300 4450 50  0001 C CNN
 F 1 "GND" V 4305 4572 50  0000 R CNN
 F 2 "" H 4300 4700 50  0001 C CNN
@@
 $EndComp
 $Comp
-L power:GND #PWR022
+L power:GND #PWR0129
 U 1 1 5EB1A73A
 P 6000 4300
-F 0 "#PWR022" H 6000 4050 50  0001 C CNN
+F 0 "#PWR0129" H 6000 4050 50  0001 C CNN
 F 1 "GND" V 6005 4172 50  0000 R CNN
 F 2 "" H 6000 4300 50  0001 C CNN
@@
 $EndComp
 $Comp
-L power:GND #PWR023
+L power:GND #PWR0130
 U 1 1 5EB1ABC9
 P 6000 4400
-F 0 "#PWR023" H 6000 4150 50  0001 C CNN
+F 0 "#PWR0130" H 6000 4150 50  0001 C CNN
 F 1 "GND" V 6005 4272 50  0000 R CNN
 F 2 "" H 6000 4400 50  0001 C CNN
@@
 $EndComp
 $Comp
-L power:GND #PWR024
+L power:GND #PWR0131
 U 1 1 5EB1B064
 P 6000 4500
-F 0 "#PWR024" H 6000 4250 50  0001 C CNN
+F 0 "#PWR0131" H 6000 4250 50  0001 C CNN
 F 1 "GND" V 6005 4372 50  0000 R CNN
 F 2 "" H 6000 4500 50  0001 C CNN
@@
 $EndComp
 $Comp
-L power:GND #PWR025
+L power:GND #PWR0132
 U 1 1 5EB1B50B
 P 6000 4600
-F 0 "#PWR025" H 6000 4350 50  0001 C CNN
+F 0 "#PWR0132" H 6000 4350 50  0001 C CNN
 F 1 "GND" V 6005 4472 50  0000 R CNN
 F 2 "" H 6000 4600 50  0001 C CNN
@@
 $EndComp
 $Comp
-L power:GND #PWR026
+L power:GND #PWR0133
 U 1 1 5EB1B9BE
 P 6000 4700
-F 0 "#PWR026" H 6000 4450 50  0001 C CNN
+F 0 "#PWR0133" H 6000 4450 50  0001 C CNN
 F 1 "GND" V 6005 4572 50  0000 R CNN
 F 2 "" H 6000 4700 50  0001 C CNN
@@
 +3.3V
 $Comp
-L power:+3.3V #PWR027
+L power:+3.3V #PWR0134
 U 1 1 5EB35B08
 P 7800 1850
-F 0 "#PWR027" H 7800 1700 50  0001 C CNN
+F 0 "#PWR0134" H 7800 1700 50  0001 C CNN
 F 1 "+3.3V" H 7815 2023 50  0000 C CNN
 F 2 "" H 7800 1850 50  0001 C CNN
@@
 +BATT
 $Comp
-L power:+5V #PWR028
+L power:+5V #PWR0135
 U 1 1 5EB368D5
 P 8250 1850
-F 0 "#PWR028" H 8250 1700 50  0001 C CNN
+F 0 "#PWR0135" H 8250 1700 50  0001 C CNN
 F 1 "+5V" H 8265 2023 50  0000 C CNN
 F 2 "" H 8250 1850 50  0001 C CNN
@@
 $EndComp
 $Comp
-L power:+BATT #PWR029
+L power:+BATT #PWR0136
 U 1 1 5EB37213
 P 8700 1850
-F 0 "#PWR029" H 8700 1700 50  0001 C CNN
+F 0 "#PWR0136" H 8700 1700 50  0001 C CNN
 F 1 "+BATT" H 8715 2023 50  0000 C CNN
 F 2 "" H 8700 1850 50  0001 C CNN
@@
 	4300 2800 4450 2800
 $Comp
-L power:GND #PWR018
+L power:GND #PWR0137
 U 1 1 5EB01534
 P 6000 3400
-F 0 "#PWR018" H 6000 3150 50  0001 C CNN
+F 0 "#PWR0137" H 6000 3150 50  0001 C CNN
 F 1 "GND" V 6005 3272 50  0000 R CNN
 F 2 "" H 6000 3400 50  0001 C CNN
@@
 $EndComp
 $Comp
-L power:GND #PWR06
+L power:GND #PWR0138
 U 1 1 5EAFEC1B
 P 4300 3600
-F 0 "#PWR06" H 4300 3350 50  0001 C CNN
+F 0 "#PWR0138" H 4300 3350 50  0001 C CNN
 F 1 "GND" V 4305 3472 50  0000 R CNN
 F 2 "" H 4300 3600 50  0001 C CNN
@@
 $EndComp
 $Comp
-L power:GND #PWR017
+L power:GND #PWR0139
 U 1 1 5EAFE4EB
 P 6000 3200
-F 0 "#PWR017" H 6000 2950 50  0001 C CNN
+F 0 "#PWR0139" H 6000 2950 50  0001 C CNN
 F 1 "GND" V 6005 3072 50  0000 R CNN
 F 2 "" H 6000 3200 50  0001 C CNN
@@
 $EndComp
 $Comp
-L power:GND #PWR016
+L power:GND #PWR0140
 U 1 1 5EAFE12E
 P 6000 3000
-F 0 "#PWR016" H 6000 2750 50  0001 C CNN
+F 0 "#PWR0140" H 6000 2750 50  0001 C CNN
 F 1 "GND" V 6005 2872 50  0000 R CNN
 F 2 "" H 6000 3000 50  0001 C CNN
@@
 $EndComp
 $Comp
-L power:+3.3V #PWR05
+L power:+3.3V #PWR0141
 U 1 1 5EAFCB48
 P 4300 3500
-F 0 "#PWR05" H 4300 3350 50  0001 C CNN
+F 0 "#PWR0141" H 4300 3350 50  0001 C CNN
 F 1 "+3.3V" V 4315 3628 50  0000 L CNN
 F 2 "" H 4300 3500 50  0001 C CNN
@@
 SPI0_nSS1
 $Comp
-L star-common-lib:CAS_stacking J1001
+L star-common-lib:CAS_stacking J5
 U 1 1 5F2F934D
 P 5150 2750
-F 0 "J1001" H 5150 3967 50  0000 C CNN
+F 0 "J5" H 5150 3967 50  0000 C CNN
 F 1 "CAS_stacking" H 5150 3876 50  0000 C CNN
 F 2 "star-common-lib:CAS_physical" H 5250 3700 50  0001 C CNN
@@
 $EndComp
 $Comp
-L star-common-lib:CAS_stacking J1001
+L star-common-lib:CAS_stacking J5
 U 2 1 5F2FC6A4
 P 5150 5150
-F 0 "J1001" H 5150 6367 50  0000 C CNN
+F 0 "J5" H 5150 6367 50  0000 C CNN
 F 1 "CAS_stacking" H 5150 6276 50  0000 C CNN
 F 2 "star-common-lib:CAS_physical" H 5250 6100 50  0001 C CNN
