File: MAX6675ISA+/MAX6675ISA+.kicad_sch (KiCad schematic)
At the start: 2 parts, among them U1301 MAX6675ISA+

Commit message: updating files to kicad 6 compatibility
Connections:
- net CS: now also U1301.6 (~{CS})
- net GND: now also U1301.1 (GND), U1301.2 (T-)
- net MISO: now also U1301.7 (SO)
- net SCK: now also U1301.5 (SCK)
- net T+: now also U1301.3 (T+)
- net VCC: now also U1301.4 (VCC)
Changed lines of the file:
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@@
-(kicad_sch (version 20210621) (generator eeschema)
+(kicad_sch (version 20211123) (generator eeschema)
   (paper "A4")
-  (junction (at 125.73 101.6) (diameter 0) (color 0 0 0 0))
-  (junction (at 176.53 88.9) (diameter 0) (color 0 0 0 0))
-  (junction (at 176.53 111.76) (diameter 0) (color 0 0 0 0))
+  (junction (at 176.53 111.76) (diameter 0) (color 0 0 0 0)
+  )
+  (junction (at 125.73 101.6) (diameter 0) (color 0 0 0 0)
+  )
+  (junction (at 176.53 88.9) (diameter 0) (color 0 0 0 0)
+  )
   (no_connect (at 129.54 106.68))
   (wire (pts (xy 125.73 101.6) (xy 124.46 101.6))
     (stroke (width 0) (type default) (color 0 0 0 0))
   )
-  (wire (pts (xy 125.73 104.14) (xy 125.73 101.6))
+  (wire (pts (xy 177.8 88.9) (xy 176.53 88.9))
     (stroke (width 0) (type default) (color 0 0 0 0))
   )
-  (wire (pts (xy 129.54 101.6) (xy 125.73 101.6))
-    (stroke (width 0) (type default) (color 0 0 0 0))
-  )
-  (wire (pts (xy 165.1 88.9) (xy 176.53 88.9))
-    (stroke (width 0) (type default) (color 0 0 0 0))
-  )
-  (wire (pts (xy 176.53 88.9) (xy 176.53 92.71))
-    (stroke (width 0) (type default) (color 0 0 0 0))
-  )
-  (wire (pts (xy 176.53 100.33) (xy 176.53 111.76))
+  (wire (pts (xy 125.73 104.14) (xy 125.73 101.6))
     (stroke (width 0) (type default) (color 0 0 0 0))
   )
@@
     (stroke (width 0) (type default) (color 0 0 0 0))
   )
-  (wire (pts (xy 177.8 88.9) (xy 176.53 88.9))
+  (wire (pts (xy 165.1 88.9) (xy 176.53 88.9))
     (stroke (width 0) (type default) (color 0 0 0 0))
+  )
+  (wire (pts (xy 176.53 100.33) (xy 176.53 111.76))
+    (stroke (width 0) (type default) (color 0 0 0 0))
+  )
+  (wire (pts (xy 129.54 101.6) (xy 125.73 101.6))
+    (stroke (width 0) (type default) (color 0 0 0 0))
+  )
+  (wire (pts (xy 176.53 88.9) (xy 176.53 92.71))
+    (stroke (width 0) (type default) (color 0 0 0 0))
+  )
+  (hierarchical_label "MISO" (shape input) (at 165.1 93.98 0)
+    (effects (font (size 1.27 1.27)) (justify left))
+  )
+  (hierarchical_label "T+" (shape input) (at 129.54 99.06 180)
+    (effects (font (size 1.27 1.27)) (justify right))
   )
   (hierarchical_label "T-" (shape input) (at 124.46 101.6 180)
     (effects (font (size 1.27 1.27)) (justify right))
+  )
+  (hierarchical_label "VCC" (shape input) (at 177.8 88.9 0)
+    (effects (font (size 1.27 1.27)) (justify left))
   )
   (hierarchical_label "CS" (shape input) (at 129.54 93.98 180)
@@
     (effects (font (size 1.27 1.27)) (justify right))
   )
-  (hierarchical_label "T+" (shape input) (at 129.54 99.06 180)
-    (effects (font (size 1.27 1.27)) (justify right))
-  )
-  (hierarchical_label "MISO" (shape input) (at 165.1 93.98 0)
-    (effects (font (size 1.27 1.27)) (justify left))
-  )
-  (hierarchical_label "VCC" (shape input) (at 177.8 88.9 0)
-    (effects (font (size 1.27 1.27)) (justify left))
-  )
-  (symbol (lib_id "power:GND") (at 125.73 104.14 0)
-    (in_bom yes) (on_board yes)
-    (property "Reference" "#PWR0106" (id 0) (at 125.73 110.49 0)
-      (effects (font (size 1.27 1.27)) hide)
-    )
-    (property "Value" "GND" (id 1) (at 125.857 108.5342 0))
-    (property "Footprint" "" (id 2) (at 125.73 104.14 0)
-      (effects (font (size 1.27 1.27)) hide)
-    )
-    (property "Datasheet" "" (id 3) (at 125.73 104.14 0)
-      (effects (font (size 1.27 1.27)) hide)
-    )
-    (pin "1")
-  )
-  (symbol (lib_id "power:GND") (at 176.53 113.03 0)
-    (in_bom yes) (on_board yes)
-    (property "Reference" "#PWR0105" (id 0) (at 176.53 119.38 0)
-      (effects (font (size 1.27 1.27)) hide)
-    )
-    (property "Value" "GND" (id 1) (at 176.657 117.4242 0))
-    (property "Footprint" "" (id 2) (at 176.53 113.03 0)
-      (effects (font (size 1.27 1.27)) hide)
-    )
-    (property "Datasheet" "" (id 3) (at 176.53 113.03 0)
-      (effects (font (size 1.27 1.27)) hide)
-    )
-    (pin "1")
-  )
-  (symbol (lib_id "Device:C") (at 176.53 96.52 0)
+  (symbol (lib_id "Device:C") (at 176.53 96.52 0) (unit 1)
     (in_bom yes) (on_board yes)
     (property "Reference" "C1301" (id 0) (at 179.451 95.3516 0)
@@
     (pin "2")
   )
-  (symbol (lib_id "star-common-lib:MAX6675ISA+") (at 147.32 101.6 0)
+  (symbol (lib_id "power:GND") (at 176.53 113.03 0) (unit 1)
     (in_bom yes) (on_board yes)
-    (property "Reference" "U1301" (id 0) (at 147.32 82.042 0))
-    (property "Value" "MAX6675ISA+" (id 1) (at 147.32 84.3534 0))
+    (property "Reference" "#PWR0105" (id 0) (at 176.53 119.38 0)
+      (effects (font (size 1.27 1.27)) hide)
+    )
+    (property "Value" "GND" (id 1) (at 176.657 117.4242 0))
+    (property "Footprint" "" (id 2) (at 176.53 113.03 0)
+      (effects (font (size 1.27 1.27)) hide)
+    )
+    (property "Datasheet" "" (id 3) (at 176.53 113.03 0)
+      (effects (font (size 1.27 1.27)) hide)
+    )
+    (pin "1")
+  )
+  (symbol (lib_id "power:GND") (at 125.73 104.14 0) (unit 1)
+    (in_bom yes) (on_board yes)
+    (property "Reference" "#PWR0106" (id 0) (at 125.73 110.49 0)
+      (effects (font (size 1.27 1.27)) hide)
+    )
+    (property "Value" "GND" (id 1) (at 125.857 108.5342 0))
+    (property "Footprint" "" (id 2) (at 125.73 104.14 0)
+      (effects (font (size 1.27 1.27)) hide)
+    )
+    (property "Datasheet" "" (id 3) (at 125.73 104.14 0)
+      (effects (font (size 1.27 1.27)) hide)
+    )
+    (pin "1")
+  )
+  (symbol (lib_id "star-common-lib:MAX6675ISA+") (at 147.32 101.6 0) (unit 1)
+    (in_bom yes) (on_board yes) (fields_autoplaced)
+    (property "Reference" "U1301" (id 0) (at 147.32 81.28 0))
+    (property "Value" "MAX6675ISA+" (id 1) (at 147.32 83.82 0))
     (property "Footprint" "star-common-lib:SOIC127P600X175-8N" (id 2) (at 147.32 101.6 0)
       (effects (font (size 1.27 1.27)) (justify left bottom) hide)
@@
       (effects (font (size 1.27 1.27)) (justify left bottom) hide)
     )
+    (pin "1")
+    (pin "2")
+    (pin "3")
+    (pin "4")
+    (pin "5")
+    (pin "6")
+    (pin "7")
+    (pin "8")
   )
   (sheet_instances
@@
       (reference "C1301") (unit 1) (value "0.1u") (footprint "Capacitor_SMD:C_0603_1608Metric")
     )
-    (path "/00000000-0000-0000-0000-000060597ca2"
+    (path "/65a8b55e-a85b-43de-a7c0-277e3d0e143e"
       (reference "U1301") (unit 1) (value "MAX6675ISA+") (footprint "star-common-lib:SOIC127P600X175-8N")
     )
